Commit message: debug gazebo spawn

File: src/mini_radi_description/urdf/mini_radi.urdf (robot description, URDF)
Before this commit: robot mini_radi, 7 links, 6 joints
Links:
- link base_link: mass None -> 5.0; geometry collision box size=1.2 0.8 0.3; visual box size=1.2 0.8 0.3
- link front_box: mass None -> 1.0; geometry collision box size=0.5 0.6 0.25; visual box size=0.5 0.6 0.25
- link left_wheel: mass None -> 0.5; geometry collision cylinder length=0.15 radius=0.22; visual cylinder length=0.15 radius=0.22
- link lidar_link: mass None -> 0.1; geometry collision cylinder length=0.08 radius=0.14; visual cylinder length=0.08 radius=0.14
- link right_wheel: mass None -> 0.5; geometry collision cylinder length=0.15 radius=0.22; visual cylinder length=0.15 radius=0.22
- link sensor_mount: mass None -> 0.2; geometry collision cylinder length=0.4 radius=0.08; visual cylinder length=0.4 radius=0.08
Joints:
- joint front_box_joint: origin xyz=0.25 0 0.275 rpy=0 0 0 -> xyz=0.45 0 0.275 rpy=0 0 0
- joint left_wheel_joint: origin xyz=0 0.48 -0.08 rpy=0 0 0 -> xyz=0 0.475 -0.08 rpy=0 0 0
- joint right_wheel_joint: origin xyz=0 -0.48 -0.08 rpy=0 0 0 -> xyz=0 -0.475 -0.08 rpy=0 0 0
- joint sensor_mount_joint: origin xyz=-0.25 0 0.35 rpy=0 0 0 -> xyz=0 0 0.35 rpy=0 0 0

Commit message: lidar sensor

File: src/mini_radi_description/urdf/mini_radi.urdf (robot description, URDF)
Before this commit: robot mini_radi, 7 links, 6 joints
Links:
- link lidar_link: mass 0.1 -> 0.2
